File: 05-technology-and-electronics/kicad/crafting-table/daughter-board/daughter-board.kicad_pcb (KiCad board)
At the start: 2 copper layers, 70 x 70 mm, 14 parts, among them J1 PN532, J10 NEO_GND_OUT, J2 To Motherboard, J3 NEO_5V_IN, J4 NEO_IN, J5 NEO_OUT, J6 NEO_GND_IN, J7 NEO_DIN, J8 NEO_DOUT, J9 NEO_5V_OUT

Commit message: updates
Parts:
- J10: value NEO_GND_OUT -> NEO_5V_OUT
- J2: value To Motherboard -> I2C to Motherboard
- J3: value NEO_5V_IN -> NEO_GND_IN
- J6: value NEO_GND_IN -> NEO_5V_IN
- J9: value NEO_5V_OUT -> NEO_GND_OUT
- moved J4 84.8 mm to (173.0, 61.1), turned to -90 degrees
- moved J2 62.8 mm to (111.0, 67.9), turned to 90 degrees
Connections:
- J1 pad 4: Net-(J1-Pin_4) -> GND
- J10 pad 1: GND -> +5V
- J2 pad 4: Net-(J1-Pin_4) -> GND
- J3 pad 1: +5V -> GND
- J6 pad 1: GND -> +5V
- J9 pad 1: +5V -> GND
Routing:
- net +5V: track 140.7 -> 78.8 mm
- net Net-(J4-Pin_3): track 24.1 -> 74.2 mm
- net Net-(J1-Pin_4): track 37.2 -> 0.00 mm
- net Net-(J1-Pin_1): track 46.3 -> 32.3 mm
- net Net-(J1-Pin_2): track 43.2 -> 36.0 mm
- net GND: track 0.00 -> 0.70 mm
Other:
- board text added: "GND"
- board text added: "SCL"
- board text added: "SDA"
- board text added: "VCC"
