File: 05-technology-and-electronics/kicad/crafting-table/daughter-board/daughter-board.kicad_sch (KiCad schematic)
At the start: 14 parts, among them J1 PN532, J10 NEO_GND_OUT, J2 I2C to Motherboard, J3 NEO_5V_IN, J4 NEO_IN, J5 NEO_OUT, J6 NEO_GND_IN, J7 NEO_DIN, J8 NEO_DOUT, J9 NEO_5V_OUT

Commit message: updates
Parts:
- J10: value NEO_GND_OUT -> NEO_5V_OUT
- J3: value NEO_5V_IN -> NEO_GND_IN
- J6: value NEO_GND_IN -> NEO_5V_IN
- J9: value NEO_5V_OUT -> NEO_GND_OUT
Connections:
- net +5V: now also J10.1 (Pin_1), J6.1 (Pin_1); no longer J3.1 (Pin_1), J9.1 (Pin_1)
- net GND: now also J1.4 (Pin_4), J2.4 (Pin_4), J3.1 (Pin_1), J9.1 (Pin_1); no longer J10.1 (Pin_1), J6.1 (Pin_1)
Changed lines of the file:
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@@
 	(paper "A4")
 	(junction
-		(at 91.44 52.07)
+		(at 96.52 67.31)
 		(diameter 0)
 		(color 0 0 0 0)
 	)
 	(junction
-		(at 96.52 71.12)
+		(at 91.44 55.88)
 		(diameter 0)
 		(color 0 0 0 0)
 	)
+	(junction
+		(at 24.13 71.12)
+		(diameter 0)
+		(color 0 0 0 0)
+	)
 	(wire
 		(pts
@@
 	(wire
 		(pts
-			(xy 90.17 55.88) (xy 96.52 55.88)
-		)
-		(stroke
-			(width 0)
-			(type default)
-		)
-	)
-	(wire
-		(pts
 			(xy 90.17 59.69) (xy 128.27 59.69)
 		)
@@
 	(wire
 		(pts
-			(xy 91.44 52.07) (xy 91.44 67.31)
+			(xy 91.44 48.26) (xy 91.44 55.88)
 		)
 		(stroke
@@
 	(wire
 		(pts
-			(xy 96.52 55.88) (xy 96.52 71.12)
+			(xy 96.52 52.07) (xy 96.52 67.31)
 		)
 		(stroke
@@
 	(wire
 		(pts
+			(xy 96.52 67.31) (xy 96.52 74.93)
+		)
+		(stroke
+			(width 0)
+			(type default)
+		)
+	)
+	(wire
+		(pts
+			(xy 91.44 71.12) (xy 90.17 71.12)
+		)
+		(stroke
+			(width 0)
+			(type default)
+		)
+	)
+	(wire
+		(pts
 			(xy 74.93 25.4) (xy 82.55 25.4)
 		)
@@
 	(wire
 		(pts
-			(xy 91.44 48.26) (xy 91.44 52.07)
-		)
-		(stroke
-			(width 0)
-			(type default)
-		)
-	)
-	(wire
-		(pts
 			(xy 128.27 59.69) (xy 128.27 57.15)
 		)
@@
 	(wire
 		(pts
-			(xy 96.52 71.12) (xy 96.52 74.93)
-		)
-		(stroke
-			(width 0)
-			(type default)
-		)
-	)
-	(wire
-		(pts
-			(xy 90.17 71.12) (xy 96.52 71.12)
+			(xy 91.44 55.88) (xy 91.44 71.12)
+		)
+		(stroke
+			(width 0)
+			(type default)
+		)
+	)
+	(wire
+		(pts
+			(xy 90.17 67.31) (xy 96.52 67.31)
+		)
+		(stroke
+			(width 0)
+			(type default)
+		)
+	)
+	(wire
+		(pts
+			(xy 90.17 52.07) (xy 96.52 52.07)
 		)
 		(stroke
@@
 	(wire
 		(pts
+			(xy 20.32 71.12) (xy 24.13 71.12)
+		)
+		(stroke
+			(width 0)
+			(type default)
+		)
+	)
+	(wire
+		(pts
 			(xy 119.38 54.61) (xy 128.27 54.61)
 		)
@@
 	(wire
 		(pts
-			(xy 91.44 67.31) (xy 90.17 67.31)
-		)
-		(stroke
-			(width 0)
-			(type default)
-		)
-	)
-	(wire
-		(pts
-			(xy 91.44 52.07) (xy 90.17 52.07)
+			(xy 90.17 55.88) (xy 91.44 55.88)
 		)
 		(stroke
@@
 			)
 		)
-		(property "Value" "NEO_GND_IN"
+		(property "Value" "NEO_5V_IN"
 			(at 74.676 56.134 0)
 			(show_name no)
@@
 	)
 	(symbol
+		(lib_id "power:GND")
+		(at 20.32 71.12 0)
+		(unit 1)
+		(body_style 1)
+		(exclude_from_sim no)
+		(in_bom yes)
+		(on_board yes)
+		(in_pos_files yes)
+		(dnp no)
+		(fields_autoplaced yes)
+		(property "Reference" "#PWR09"
+			(at 20.32 77.47 0)
+			(hide yes)
+			(show_name no)
+			(do_not_autoplace no)
+			(effects
+				(font
+					(size 1.27 1.27)
+				)
+			)
+		)
+		(property "Value" "GND"
+			(at 20.32 76.2 0)
+			(show_name no)
+			(do_not_autoplace no)
+			(effects
+				(font
+					(size 1.27 1.27)
+				)
+			)
+		)
+		(property "Footprint" ""
+			(at 20.32 71.12 0)
+			(hide yes)
+			(show_name no)
+			(do_not_autoplace no)
+			(effects
+				(font
+					(size 1.27 1.27)
+				)
+			)
+		)
+		(property "Datasheet" ""
+			(at 20.32 71.12 0)
+			(hide yes)
+			(show_name no)
+			(do_not_autoplace no)
+			(effects
+				(font
+					(size 1.27 1.27)
+				)
+			)
+		)
+		(property "Description" "Power symbol creates a global label with name \"GND\" , ground"
+			(at 20.32 71.12 0)
+			(hide yes)
+			(show_name no)
+			(do_not_autoplace no)
+			(effects
+				(font
+					(size 1.27 1.27)
+				)
+			)
+		)
+		(pin "1"
+		)
+		(instances
+			(project "daughter-board"
+				(path "/f9b1fd56-0a6e-444d-931e-42cdc1495419"
+					(reference "#PWR09")
+					(unit 1)
+				)
+			)
+		)
+	)
+	(symbol
 		(lib_id "Mechanical:MountingHole")
 		(at 44.45 100.33 0)
@@
 			)
 		)
-		(property "Value" "NEO_GND_OUT"
+		(property "Value" "NEO_5V_OUT"
 			(at 73.66 71.12 0)
 			(show_name no)
@@
 			)
 		)
-		(property "Value" "NEO_5V_OUT"
+		(property "Value" "NEO_GND_OUT"
 			(at 74.422 67.31 0)
 			(show_name no)
@@
 			)
 		)
-		(property "Value" "NEO_5V_IN"
+		(property "Value" "NEO_GND_IN"
 			(at 75.438 52.07 0)
 			(show_name no)
