File: 05-technology-and-electronics/kicad/crafting-table/motherboard/motherboard.kicad_pcb (KiCad board)
At the start: 2 copper layers, 123.6 x 86.4 mm, 38 parts, among them J1 Barrel_Jack, J10 SLOT6_I2C, J11 SLOT7_I2C, J12 SLOT8_I2C, J13 NEOPIXEL_OUT, J14 SERVO_0, J15 SERVO_1, J16 SERVO_2, J17 DFPlayer_L, J18 DFPlayer_R, J19 PCA9548A_0_L, J2 ESP32_L, J20 PCA9548A_0_R, J21 PCA9548A_1_L, J22 PCA9548A_1_R, J23 SPEAKER, J24 CAPACITIVE, J25 VIBRATION, J26 EXTRA_PINS, J3 ESP32_R, J4 SLOT0_I2C, J5 SLOT1_I2C, J6 SLOT2_I2C, J7 SLOT3_I2C, J8 SLOT4_I2C, J9 SLOT5_I2C, Q1 2N7002

Commit message: updates
Parts:
- J23, J24, J25: footprint TerminalBlock_Phoenix:TerminalBlock_Phoenix_MKDS-3-2-5.08_1x02_P5.08mm_Horizontal -> TerminalBlock_TE-Connectivity:TerminalBlock_TE_282834-2_1x02_P2.54mm_Horizontal
- Q1: value 2N7002 -> Q_NMOS_GDS
- moved C1 2.94 mm to (146.9, 63.5)
- moved Q1 0.29 mm to (100.6, 85.8)
Connections:
- J10 pad 1: +5V -> Net-(J10-Pin_1)
- J10 pad 2: GND -> Net-(J10-Pin_2)
- J10 pad 3: Net-(J10-Pin_3) -> +5V
- J10 pad 4: Net-(J10-Pin_4) -> GND
- J11 pad 1: +5V -> Net-(J11-Pin_1)
- J11 pad 2: GND -> Net-(J11-Pin_2)
- J11 pad 3: Net-(J11-Pin_3) -> +5V
- J11 pad 4: Net-(J11-Pin_4) -> GND
- J12 pad 1: +5V -> Net-(J12-Pin_1)
- J12 pad 2: GND -> Net-(J12-Pin_2)
- J12 pad 3: Net-(J12-Pin_3) -> +5V
- J12 pad 4: Net-(J12-Pin_4) -> GND
- J19 pad 10: Net-(J11-Pin_4) -> Net-(J11-Pin_1)
- J19 pad 11: Net-(J10-Pin_3) -> Net-(J10-Pin_2)
- J19 pad 12: Net-(J10-Pin_4) -> Net-(J10-Pin_1)
- J19 pad 9: Net-(J11-Pin_3) -> Net-(J11-Pin_2)
- J21 pad 10: Net-(J12-Pin_4) -> Net-(J12-Pin_1)
- J21 pad 9: Net-(J12-Pin_3) -> Net-(J12-Pin_2)
- J4 pad 1: +5V -> Net-(J20-Pin_1)
- J4 pad 2: GND -> Net-(J20-Pin_2)
- J4 pad 3: Net-(J20-Pin_2) -> +5V
- J4 pad 4: Net-(J20-Pin_1) -> GND
- J5 pad 1: +5V -> Net-(J20-Pin_3)
- J5 pad 2: GND -> Net-(J20-Pin_4)
- J5 pad 3: Net-(J20-Pin_4) -> +5V
- J5 pad 4: Net-(J20-Pin_3) -> GND
- J6 pad 1: +5V -> Net-(J20-Pin_5)
- J6 pad 2: GND -> Net-(J20-Pin_6)
- J6 pad 3: Net-(J20-Pin_6) -> +5V
- J6 pad 4: Net-(J20-Pin_5) -> GND
- J7 pad 1: +5V -> Net-(J20-Pin_7)
- J7 pad 2: GND -> Net-(J20-Pin_8)
- J7 pad 3: Net-(J20-Pin_8) -> +5V
- J7 pad 4: Net-(J20-Pin_7) -> GND
- J8 pad 1: +5V -> Net-(J20-Pin_11)
- J8 pad 2: GND -> Net-(J20-Pin_12)
- J8 pad 3: Net-(J20-Pin_11) -> +5V
- J8 pad 4: Net-(J20-Pin_12) -> GND
- J9 pad 1: +5V -> Net-(J20-Pin_9)
- J9 pad 2: GND -> Net-(J20-Pin_10)
- J9 pad 3: Net-(J20-Pin_9) -> +5V
- J9 pad 4: Net-(J20-Pin_10) -> GND
- Q1 pad 2: GND -> Net-(D1-A)
- Q1 pad 3: Net-(D1-A) -> GND
Routing:
- net +5V: track 354.4 -> 567.8 mm
- net Net-(J11-Pin_4): track 36.9 -> 0.00 mm
- net Net-(J11-Pin_2): track 0.00 -> 35.4 mm
- net Net-(J11-Pin_3): track 35.2 -> 0.00 mm
- net Net-(J11-Pin_1): track 0.00 -> 28.2 mm
- net Net-(J12-Pin_3): track 25.0 -> 0.00 mm
- net Net-(J12-Pin_4): track 24.6 -> 0.00 mm
- net Net-(J10-Pin_4): track 23.9 -> 0.00 mm
- net Net-(J10-Pin_3): track 22.8 -> 0.00 mm
- net Net-(J10-Pin_2): track 0.00 -> 22.7 mm
- net Net-(J12-Pin_2): track 0.00 -> 22.6 mm
- net Net-(J12-Pin_1): track 0.00 -> 16.6 mm
- net Net-(J10-Pin_1): track 0.00 -> 16.0 mm
- net Net-(D1-A): track 33.8 -> 23.5 mm
- net Net-(J20-Pin_1): track 22.9 -> 13.7 mm
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