File: 05-technology-and-electronics/kicad/crafting-table/motherboard/motherboard.kicad_sch (KiCad schematic)
At the start: 38 parts, among them J1 Barrel_Jack, J10 SLOT6_I2C, J11 SLOT7_I2C, J12 SLOT8_I2C, J13 NEOPIXEL_OUT, J14 SERVO_0, J15 SERVO_1, J16 SERVO_2, J17 DFPlayer_L, J18 DFPlayer_R, J19 PCA9548A_0_L, J2 ESP32_L, J20 PCA9548A_0_R, J21 PCA9548A_1_L, J22 PCA9548A_1_R, J23 SPEAKER, J24 CAPACITIVE, J25 VIBRATION, J26 EXTRA_PINS, J3 ESP32_R, J4 SLOT0_I2C, J5 SLOT1_I2C, J6 SLOT2_I2C, J7 SLOT3_I2C, J8 SLOT4_I2C, J9 SLOT5_I2C, Q1 2N7002

Commit message: updates
Parts:
- removed Q1: 2N7002, Package_TO_SOT_THT:TO-220-3_Vertical, symbol Transistor_FET:2N7002
- added Q1: Q_NMOS_GDS, Package_TO_SOT_THT:TO-220-3_Vertical, symbol Transistor_FET:Q_NMOS_GDS
- J23, J24, J25: footprint TerminalBlock_Phoenix:TerminalBlock_Phoenix_MKDS-3-2-5.08_1x02_P5.08mm_Horizontal -> TerminalBlock_TE-Connectivity:TerminalBlock_TE_282834-2_1x02_P2.54mm_Horizontal
Connections:
- net +5V: now also J10.3 (Pin_3), J11.3 (Pin_3), J12.3 (Pin_3), J4.3 (Pin_3), J5.3 (Pin_3), J6.3 (Pin_3), J7.3 (Pin_3), J8.3 (Pin_3), J9.3 (Pin_3); no longer J10.1 (Pin_1), J11.1 (Pin_1), J12.1 (Pin_1), J4.1 (Pin_1), J5.1 (Pin_1), J6.1 (Pin_1), J7.1 (Pin_1), J8.1 (Pin_1), J9.1 (Pin_1)
- net GND: now also J10.4 (Pin_4), J11.4 (Pin_4), J12.4 (Pin_4), J4.4 (Pin_4), J5.4 (Pin_4), J6.4 (Pin_4), J7.4 (Pin_4), J8.4 (Pin_4), J9.4 (Pin_4), Q1.3 (S); no longer J10.2 (Pin_2), J11.2 (Pin_2), J12.2 (Pin_2), J4.2 (Pin_2), J5.2 (Pin_2), J6.2 (Pin_2), J7.2 (Pin_2), J8.2 (Pin_2), J9.2 (Pin_2)
- net at J20.6 (Pin_6): now also J6.2 (Pin_2); no longer J6.3 (Pin_3)
- net at J20.5 (Pin_5): now also J6.1 (Pin_1); no longer J6.4 (Pin_4)
- net at J20.9 (Pin_9): now also J9.1 (Pin_1); no longer J9.3 (Pin_3)
- net at J20.10 (Pin_10): now also J9.2 (Pin_2); no longer J9.4 (Pin_4)
- net at J20.1 (Pin_1): now also J4.1 (Pin_1); no longer J4.4 (Pin_4)
- net at J20.11 (Pin_11): now also J8.1 (Pin_1); no longer J8.3 (Pin_3)
- net at J20.12 (Pin_12): now also J8.2 (Pin_2); no longer J8.4 (Pin_4)
- net at J20.2 (Pin_2): now also J4.2 (Pin_2); no longer J4.3 (Pin_3)
- net at J20.3 (Pin_3): now also J5.1 (Pin_1); no longer J5.4 (Pin_4)
- net at J20.4 (Pin_4): now also J5.2 (Pin_2); no longer J5.3 (Pin_3)
- net at J20.7 (Pin_7): now also J7.1 (Pin_1); no longer J7.4 (Pin_4)
- net at J20.8 (Pin_8): now also J7.2 (Pin_2); no longer J7.3 (Pin_3)
- net at D1.2 (A), J25.1 (Pin_1): now also Q1.2 (D)
- net at J19.9 (Pin_9): now also J11.2 (Pin_2); no longer J11.3 (Pin_3)
- net at J19.10 (Pin_10): now also J11.1 (Pin_1); no longer J11.4 (Pin_4)
- net at J19.11 (Pin_11): now also J10.2 (Pin_2); no longer J10.3 (Pin_3)
- net at J19.12 (Pin_12): now also J10.1 (Pin_1); no longer J10.4 (Pin_4)
- net at J21.9 (Pin_9): now also J12.2 (Pin_2); no longer J12.3 (Pin_3)
- net at J21.10 (Pin_10): now also J12.1 (Pin_1); no longer J12.4 (Pin_4)
- net at J2.9 (Pin_9), R5.1: now also Q1.1 (G)
